Commit message: body and segment part were finished, both rviz and gazebo launch files were written

File: strirus_robot_description/urdf/materials.xacro (robot description, xacro)
@@ -1,28 +1,28 @@
 <?xml version="1.0"?>
 <robot>
-<!-- Import Rviz colors -->
-  <material name="black">
-    <color rgba="0.0 0.0 0.0 1.0"/>
-  </material>
-  <material name="blue">
-    <color rgba="0.0 0.0 0.8 1.0"/>
-  </material>
-  <material name="green">
-    <color rgba="0.0 0.8 0.0 1.0"/>
-  </material>
-  <material name="grey">
-    <color rgba="0.2 0.2 0.2 1.0"/>
-  </material>
-  <material name="orange">
-    <color rgba="${255/255} ${108/255} ${10/255} 1.0"/>
-  </material>
-  <material name="brown">
-    <color rgba="${222/255} ${207/255} ${195/255} 1.0"/>
-  </material>
-  <material name="red">
-    <color rgba="0.8 0.0 0.0 1.0"/>
-  </material>
-  <material name="white">
-    <color rgba="1.0 1.0 1.0 1.0"/>
-  </material>
+    <!-- Import Rviz colors -->
+    <material name="black">
+        <color rgba="0.0 0.0 0.0 1.0"/>
+    </material>
+    <material name="blue">
+        <color rgba="0.0 0.0 0.8 1.0"/>
+    </material>
+    <material name="green">
+        <color rgba="0.0 0.8 0.0 1.0"/>
+    </material>
+    <material name="grey">
+        <color rgba="0.2 0.2 0.2 1.0"/>
+    </material>
+    <material name="orange">
+        <color rgba="${255/255} ${108/255} ${10/255} 1.0"/>
+    </material>
+    <material name="brown">
+        <color rgba="${222/255} ${207/255} ${195/255} 1.0"/>
+    </material>
+    <material name="red">
+        <color rgba="0.8 0.0 0.0 1.0"/>
+    </material>
+    <material name="white">
+        <color rgba="1.0 1.0 1.0 1.0"/>
+    </material>
 </robot>

File: strirus_robot_description/urdf/strirus_gamma.urdf (robot description, URDF)
Before this commit: robot Strirus_gamma, 5 links, 4 joints
Links:
- removed link base_link
- added link base_footprint
- link body_1_part: geometry collision mesh filename=package://strirus_cad_design/stl/collision/body_1_15_part.s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 scale=1 1 1; visual mesh filename=package://strirus_cad_design/stl/visual/body_1_15_part.stl scale=1 1 1
- link body_2_part: geometry collision mesh filename=package://strirus_cad_design/stl/collision/body_2_15_part.s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 scale=1 1 1; visual mesh filename=package://strirus_cad_design/stl/visual/body_2_15_part.stl scale=1 1 1
- link bridge_1_part: geometry collision mesh filename=package://strirus_cad_design/stl/collision/bridge_1_part.stl scale=1 1 1; visual mesh filename=package://strirus_cad_design/stl/visual/bridge_1_part.stl scale=1 1 1
- link bridge_2_part: geometry collision mesh filename=package://strirus_cad_design/stl/collision/bridge_2_part.stl scale=1 1 1; visual mesh filename=package://strirus_cad_design/stl/visual/bridge_2_part.stl scale=1 1 1
Joints:
- removed joint base_link_body_1_part_fixed
- removed joint body_1_part_bridge_1_part_fixed
- removed joint bridge_1_part_bridge_2_part_revolute
- added joint base_footprint_body_1_part_fixed: type fixed, parent base_footprint, child body_1_part, origin xyz=0 0 0.055 rpy=0  0  0
- joint bridge_2_part_body_2_part_fixed: origin (none) -> xyz=0.03 0 0 rpy=0 0 0

File: strirus_robot_description/urdf/strirus_gamma.xacro (robot description, xacro)
@@ -1,69 +1,75 @@
 <?xml version="1.0"?>
-<robot name="Strirus_gamma" xmlns:xacro="http://www.ros.org/wiki/xacro">
-	<gazebo>
-		<self_collide> 1 </self_collide>
-	</gazebo>
-<!-- 	<xacro:arg name="namespace" default="/"/>
-	<xacro:property name="namespace" value="$(arg namespace)" /> -->
-	<!-- Some constants -->
-	<xacro:property name="deg2rad" value="${pi / 180}" />
-	<xacro:property name="rad2deg" value="${180 / pi}" />
-    <xacro:property name="number_of_legs" value="${6 - 1}" />
-	<!-- Constants for simulating -->
-	<!-- Xacro arg provides xacro.py file.xacro real_number_of_legs:=12 -->
-	<!-- simulation  options-->
-	<xacro:arg name="ideal_motors" default="0" doc="0 - no, 1 - yes"/>
-	<xacro:arg name="ideal_segment_joint" default="0" doc="0 - no, 1 - yes"/>
-	<xacro:arg name="leg_fancy_physics" default="0" doc="0 - no, 1 - yes"/>
-	<!-- omni-directional -->
-	<xacro:arg name="omni_angle" default="30" doc="possible angles 0,15,30,45"/>
-	<!-- leg size -->
-	<xacro:arg name="leg_size" default="0" doc="0 - 55, 1 - 70"/>
-	<!-- angle between legs -->
-	<xacro:arg name="angle_btw_legs" default="0" doc="in degrees, or 'specific' for choosing specific angle for each leg (cclock)"/>
-	<xacro:arg name="offset_btw_legs_wave" default="0" doc="in degrees"/>
-	<xacro:arg name="l_specific_angle_btw_legs" default="[0,0,0,0,0,0]" doc=""/>
-	<xacro:arg name="r_specific_angle_btw_legs" default="[0,0,0,0,0,0]" doc=""/>
-	<!-- segmentation -->
-	<xacro:arg name="segment_dof" default="1up" doc="possible '0','1up','1side','2'"/>
-	<xacro:arg name="up_segment_angle" default="0" doc="in degrees"/>
-	<xacro:arg name="side_segment_angle" default="0" doc="in degrees"/>
-	<!-- arg to properties with converting to rad if it is needed -->
-	<!-- simulation  options-->
-	<xacro:property name="ideal_motors" value="$(arg ideal_motors)"/>
-	<xacro:property name="ideal_segment_joint" value="$(arg ideal_segment_joint)"/>
-	<xacro:property name="leg_fancy_physics" value="$(arg leg_fancy_physics)"/>
-	<!-- omni-directional -->
-	<xacro:property name="omni_angle" value="$(arg omni_angle)"/>
-	<!-- leg size -->
-	<xacro:property name="leg_size" value="$(arg leg_size)"/>
-	<!-- angle between legs -->
-	<xacro:property name="angle_btw_legs" value="$(arg angle_btw_legs)"/>
-	<xacro:if value="${str(angle_btw_legs) == 'specific'}">
-		<xacro:property name="l_specific_angle_btw_legs" value="$(arg l_specific_angle_btw_legs)"/>
-		<xacro:property name="r_specific_angle_btw_legs" value="$(arg r_specific_angle_btw_legs)"/>
-		<xacro:property name="offset_btw_legs_wave" value="0"/>
-	</xacro:if>
-	<xacro:if value="${str(angle_btw_legs) != 'specific'}">
-		<xacro:property name="offset_btw_legs_wave" value="$(arg offset_btw_legs_wave)"/>
-	</xacro:if>
-	<!-- segmentation -->
-	<xacro:property name="segment_dof" value="$(arg segment_dof)"/>
-	<xacro:property name="up_segment_angle" value="$(arg up_segment_angle)"/>
-	<xacro:property name="side_segment_angle" value="$(arg side_segment_angle)"/>
-	<!-- Needed constants-variables -->
-	<xacro:property name="dist_btw_legs" value="${0.13}" />
-	<xacro:property name="robot_height_center" value="${0.025}" />
-	<xacro:property name="dist_btw_body_origins" value="${0.554}" />
-	<xacro:property name="dist_btw_bridge_holdings" value="${0.06}" />
-	<xacro:property name="dist_origin_1bridge_hole" value="${0.247}" />
-	<xacro:property name="dist_origin_bridge_center" value="${0.277}" />
-	<xacro:property name="dist_origin_2bridge_hole" value="${0.307}" />
-<!-- includes parts -->
-		<!-- Import all Gazebo-customization elements, including Gazebo colors -->
-	<!-- <xacro:include filename="$(find strirus_robot_description)/urdf/strirus_plugins.gazebo" /> -->
-	<!-- Import Rviz colors -->
-	<xacro:include filename="$(find strirus_robot_description)/urdf/materials.xacro" />
-	<xacro:include filename="$(find strirus_robot_description)/urdf/strirus_gamma_body_bridge.xacro" />
-	<xacro:include filename="$(find strirus_robot_description)/urdf/strirus_gamma_legs.xacro" />
+<robot name="strirus_gamma" xmlns:xacro="http://www.ros.org/wiki/xacro">
+    <gazebo>
+        <self_collide>1</self_collide>
+    </gazebo>
+    <!-- 	<xacro:arg name="namespace" default="/"/>
+        <xacro:property name="namespace" value="$(arg namespace)" /> -->
+    <!-- Some constants -->
+    <xacro:property name="deg2rad" value="${pi / 180}"/>
+    <xacro:property name="rad2deg" value="${180 / pi}"/>
+    <xacro:property name="number_of_legs" value="${6 - 1}"/>
+    <!-- Constants for simulating -->
+    <!-- Xacro arg provides xacro.py file.xacro real_number_of_legs:=12 -->
+    <!-- simulation  options-->
+    <xacro:arg name="ideal_motors" default="0" doc="0 - no, 1 - yes"/>
+    <xacro:arg name="ideal_segment_joint" default="0" doc="0 - no, 1 - yes"/>
+    <xacro:arg name="leg_fancy_physics" default="0" doc="0 - no, 1 - yes"/>
+    <!-- omni-directional -->
+    <xacro:arg name="omni_angle" default="15" doc="possible angles 0,15,30,45"/>
+    <!-- leg size -->
+    <xacro:arg name="leg_height" default="0" doc="0 - 55, 1 - 70"/>
+    <!-- angle between legs -->
+    <xacro:arg name="angle_btw_legs" default="0"
+               doc="in degrees, or 'specific' for choosing specific angle for each leg (cclock)"/>
+    <xacro:arg name="offset_btw_legs_wave" default="0" doc="in degrees"/>
+    <xacro:arg name="l_specific_angle_btw_legs" default="[0,0,0,0,0,0]" doc=""/>
+    <xacro:arg name="r_specific_angle_btw_legs" default="[0,0,0,0,0,0]" doc=""/>
+    <!-- segmentation -->
+    <xacro:arg name="segment_dof" default="2" doc="possible '0','1up','1side','2'"/>
+    <xacro:arg name="up_segment_angle" default="0" doc="in degrees"/>
+    <xacro:arg name="side_segment_angle" default="0" doc="in degrees"/>
+    <!-- arg to properties with converting to rad if it is needed -->
+    <!-- simulation  options-->
+    <xacro:property name="ideal_motors" value="$(arg ideal_motors)"/>
+    <xacro:property name="ideal_segment_joint" value="$(arg ideal_segment_joint)"/>
+    <xacro:property name="leg_fancy_physics" value="$(arg leg_fancy_physics)"/>
+    <!-- omni-directional -->
+    <xacro:property name="omni_angle" value="$(arg omni_angle)"/>
+    <!-- leg size -->
+    <xacro:property name="leg_height" value="$(arg leg_height)"/>
+    <xacro:if value="${leg_height == 1}">
+        <xacro:property name="leg_height" value="${0.07}"/>
+    </xacro:if>
+    <xacro:if value="${leg_height == 0}">
+        <xacro:property name="leg_height" value="${0.055}"/>
+    </xacro:if>
+    <!-- angle between legs -->
+    <xacro:property name="angle_btw_legs" value="$(arg angle_btw_legs)"/>
+    <xacro:if value="${str(angle_btw_legs) == 'specific'}">
+        <xacro:property name="l_specific_angle_btw_legs" value="$(arg l_specific_angle_btw_legs)"/>
+        <xacro:property name="r_specific_angle_btw_legs" value="$(arg r_specific_angle_btw_legs)"/>
+        <xacro:property name="offset_btw_legs_wave" value="0"/>
+    </xacro:if>
+    <xacro:if value="${str(angle_btw_legs) != 'specific'}">
+        <xacro:property name="offset_btw_legs_wave" value="$(arg offset_btw_legs_wave)"/>
+    </xacro:if>
+    <!-- segmentation -->
+    <xacro:property name="segment_dof" value="$(arg segment_dof)"/>
+    <xacro:property name="up_segment_angle" value="$(arg up_segment_angle)"/>
+    <xacro:property name="side_segment_angle" value="$(arg side_segment_angle)"/>
+    <!-- Needed constants-variables -->
+    <xacro:property name="dist_btw_legs" value="${0.13}"/>
+    <xacro:property name="dist_btw_body_origins" value="${0.554}"/>
+    <xacro:property name="dist_body_1_bridge_1" value="${0.247}"/>
+    <xacro:property name="dist_bridge_1_bridge_2" value="${0.03}"/>
+    <xacro:property name="dist_bridge_2_body_2" value="${0.03}"/>
+    <xacro:property name="dist_body_2_leg_count_point" value="${0.247}"/>
+    <!-- includes parts -->
+    <!-- Import all Gazebo-customization elements, including Gazebo colors -->
+    <!-- <xacro:include filename="$(find strirus_robot_description)/urdf/strirus_plugins.gazebo" /> -->
+    <!-- Import Rviz colors -->
+    <xacro:include filename="$(find strirus_robot_description)/urdf/materials.xacro"/>
+    <xacro:include filename="$(find strirus_robot_description)/urdf/strirus_gamma_body_bridge.xacro"/>
+    <xacro:include filename="$(find strirus_robot_description)/urdf/strirus_gamma_legs.xacro"/>
 </robot>
