Commit message: temp commit

File: strirus_robot_description/urdf/strirus_gamma.xacro (robot description, xacro)
@@ -1,4 +1,9 @@
 <?xml version="1.0"?>
 <robot name="strirus_gamma" xmlns:xacro="http://www.ros.org/wiki/xacro">
+    <mujoco>
+	<!-- if it doesn't work, try this and put the value by your own
+		$(find strirus_cad_design)/stl/collision-->
+        <compiler meshdir="../../../../strirus_cad_design/stl/collision/" balanceinertia="true" inertiafromgeom="false" convexhull="false" fusestatic="false"/>
+    </mujoco>
     <gazebo>
         <self_collide>1</self_collide>

File: strirus_robot_description/urdf/strirus_gamma_legs.xacro (robot description, xacro)
@@ -90,5 +90,5 @@
             </xacro:if>
             <axis xyz="0 -1  0"/>
-            <limit effort="1.5" lower="-1e+100" upper="1e+100" velocity="3.0"/>
+            <limit effort="1.5" lower="-1e+5" upper="1e+5" velocity="3.0"/>
             <xacro:if value="${ideal_leg_motors == 1}">
                 <joint_properties damping="0.0" friction="0.0"/>
