Commit message: temp commit. Refactoring + some part of leg's code was done

File: strirus_robot_description/urdf/strirus_gamma.urdf (robot description, URDF)
Before this commit: robot strirus_gamma, 5 links, 2 joints
Links:
- added link leg_left_0, mass 0.010307884; collision mesh filename=package://strirus_cad_design/stl/collision/leg_55.stl scale=1 1 1; visual mesh filename=package://strirus_cad_design/stl/visual/leg_55.stl scale=1 1 1
- added link leg_left_1, mass 0.010307884; collision mesh filename=package://strirus_cad_design/stl/collision/leg_55.stl scale=1 1 1; visual mesh filename=package://strirus_cad_design/stl/visual/leg_55.stl scale=1 1 1
- added link leg_left_2, mass 0.010307884; collision mesh filename=package://strirus_cad_design/stl/collision/leg_55.stl scale=1 1 1; visual mesh filename=package://strirus_cad_design/stl/visual/leg_55.stl scale=1 1 1
- added link leg_left_3, mass 0.010307884; collision mesh filename=package://strirus_cad_design/stl/collision/leg_55.stl scale=1 1 1; visual mesh filename=package://strirus_cad_design/stl/visual/leg_55.stl scale=1 1 1
- added link leg_left_4, mass 0.010307884; collision mesh filename=package://strirus_cad_design/stl/collision/leg_55.stl scale=1 1 1; visual mesh filename=package://strirus_cad_design/stl/visual/leg_55.stl scale=1 1 1
- added link leg_left_5, mass 0.010307884; collision mesh filename=package://strirus_cad_design/stl/collision/leg_55.stl scale=1 1 1; visual mesh filename=package://strirus_cad_design/stl/visual/leg_55.stl scale=1 1 1
- added link leg_right_0, mass 0.010307884; collision mesh filename=package://strirus_cad_design/stl/collision/leg_55.stl scale=1 1 1; visual mesh filename=package://strirus_cad_design/stl/visual/leg_55.stl scale=1 1 1
- added link leg_right_1, mass 0.010307884; collision mesh filename=package://strirus_cad_design/stl/collision/leg_55.stl scale=1 1 1; visual mesh filename=package://strirus_cad_design/stl/visual/leg_55.stl scale=1 1 1
- added link leg_right_2, mass 0.010307884; collision mesh filename=package://strirus_cad_design/stl/collision/leg_55.stl scale=1 1 1; visual mesh filename=package://strirus_cad_design/stl/visual/leg_55.stl scale=1 1 1
- added link leg_right_3, mass 0.010307884; collision mesh filename=package://strirus_cad_design/stl/collision/leg_55.stl scale=1 1 1; visual mesh filename=package://strirus_cad_design/stl/visual/leg_55.stl scale=1 1 1
- added link leg_right_4, mass 0.010307884; collision mesh filename=package://strirus_cad_design/stl/collision/leg_55.stl scale=1 1 1; visual mesh filename=package://strirus_cad_design/stl/visual/leg_55.stl scale=1 1 1
- added link leg_right_5, mass 0.010307884; collision mesh filename=package://strirus_cad_design/stl/collision/leg_55.stl scale=1 1 1; visual mesh filename=package://strirus_cad_design/stl/visual/leg_55.stl scale=1 1 1
- link body_1_part: geometry collision mesh filename=package://strirus_cad_design/stl/collision/body_1_0_part.stl scale=1 1 1; visual mesh filename=package://strirus_cad_design/stl/visual/body_1_0_part.stl scale=1 1 1
- link body_2_part: geometry collision mesh filename=package://strirus_cad_design/stl/collision/body_2_0_part.stl scale=1 1 1; visual mesh filename=package://strirus_cad_design/stl/visual/body_2_0_part.stl scale=1 1 1
Joints:
- added joint body_1_part_bridge_1_part_revolute: type revolute, parent body_1_part, child bridge_1_part, origin xyz=0.247 0 0 rpy=0       0      0, axis 0 0  -1, limit lower=-0.261799387799 upper=0.261799387799 effort=30 velocity=5
- added joint bridge_1_part_bridge_2_part_revolute: type revolute, parent bridge_1_part, child bridge_2_part, origin xyz=0.03 0 0 rpy=0       0      0, axis 0 -1  0, limit lower=-1.308996939 upper=1.308996939 effort=30 velocity=5
- added joint leg_left_0_revolute_joint: type revolute, parent body_1_part, child leg_left_0, origin xyz=0.0 0.1345  0 rpy=0       0      0, axis 0 1  0, limit lower=-1e+100 upper=1e+100 effort=30 velocity=3.0
- added joint leg_left_1_revolute_joint: type revolute, parent body_1_part, child leg_left_1, origin xyz=0.13 0.1515  0 rpy=0       0      0, axis 0 1  0, limit lower=-1e+100 upper=1e+100 effort=30 velocity=3.0
- added joint leg_left_2_revolute_joint: type revolute, parent body_1_part, child leg_left_2, origin xyz=0.26 0.1345  0 rpy=0       0      0, axis 0 1  0, limit lower=-1e+100 upper=1e+100 effort=30 velocity=3.0
- added joint leg_left_3_revolute_joint: type revolute, parent body_2_part, child leg_left_3, origin xyz=0.247 0.1515  0 rpy=0       0      0, axis 0 1  0, limit lower=-1e+100 upper=1e+100 effort=30 velocity=3.0
- added joint leg_left_4_revolute_joint: type revolute, parent body_2_part, child leg_left_4, origin xyz=0.117 0.1345  0 rpy=0       0      0, axis 0 1  0, limit lower=-1e+100 upper=1e+100 effort=30 velocity=3.0
- added joint leg_left_5_revolute_joint: type revolute, parent body_2_part, child leg_left_5, origin xyz=-0.013 0.1515  0 rpy=0       0      0, axis 0 1  0, limit lower=-1e+100 upper=1e+100 effort=30 velocity=3.0
- added joint leg_right_0_revolute_joint: type revolute, parent body_1_part, child leg_right_0, origin xyz=0.0 -0.1345  0 rpy=0       0      0, axis 0 1  0, limit lower=-1e+100 upper=1e+100 effort=30 velocity=3.0
- added joint leg_right_1_revolute_joint: type revolute, parent body_1_part, child leg_right_1, origin xyz=0.13 -0.1515  0 rpy=0       0      0, axis 0 1  0, limit lower=-1e+100 upper=1e+100 effort=30 velocity=3.0
- added joint leg_right_2_revolute_joint: type revolute, parent body_1_part, child leg_right_2, origin xyz=0.26 -0.1345  0 rpy=0       0      0, axis 0 1  0, limit lower=-1e+100 upper=1e+100 effort=30 velocity=3.0
- added joint leg_right_3_revolute_joint: type revolute, parent body_2_part, child leg_right_3, origin xyz=0.247 -0.1515  0 rpy=0       0      0, axis 0 1  0, limit lower=-1e+100 upper=1e+100 effort=30 velocity=3.0
- added joint leg_right_4_revolute_joint: type revolute, parent body_2_part, child leg_right_4, origin xyz=0.117 -0.1345  0 rpy=0       0      0, axis 0 1  0, limit lower=-1e+100 upper=1e+100 effort=30 velocity=3.0
- added joint leg_right_5_revolute_joint: type revolute, parent body_2_part, child leg_right_5, origin xyz=-0.013 -0.1515  0 rpy=0       0      0, axis 0 1  0, limit lower=-1e+100 upper=1e+100 effort=30 velocity=3.0

File: strirus_robot_description/urdf/strirus_gamma.xacro (robot description, xacro)
@@ -10,4 +10,5 @@
     <xacro:property name="rad2deg" value="${180 / pi}"/>
     <xacro:property name="number_of_legs" value="${6 - 1}"/>
+    <xacro:property name="amount_of_legs_one_part" value="${3}"/>
     <!-- Constants for simulating -->
     <!-- Xacro arg provides xacro.py file.xacro real_number_of_legs:=12 -->
@@ -17,13 +18,14 @@
     <xacro:arg name="leg_fancy_physics" default="0" doc="0 - no, 1 - yes"/>
     <!-- omni-directional -->
-    <xacro:arg name="omni_angle" default="15" doc="possible angles 0,15,30,45"/>
+    <xacro:arg name="omni_angle" default="0" doc="possible angles 0,15,30,45"/>
     <!-- leg size -->
     <xacro:arg name="leg_height" default="0" doc="0 - 55, 1 - 70"/>
     <!-- angle between legs -->
-    <xacro:arg name="angle_btw_legs" default="0"
+    <xacro:arg name="angle_btw_legs" default="specific"
                doc="in degrees, or 'specific' for choosing specific angle for each leg (cclock)"/>
-    <xacro:arg name="offset_btw_legs_wave" default="0" doc="in degrees"/>
-    <xacro:arg name="l_specific_angle_btw_legs" default="[0,0,0,0,0,0]" doc=""/>
-    <xacro:arg name="r_specific_angle_btw_legs" default="[0,0,0,0,0,0]" doc=""/>
+    <xacro:arg name="angle_for_0_l_leg" default="0" doc="in degrees"/>
+    <xacro:arg name="angle_for_0_r_leg" default="4" doc="in degrees"/>
+    <xacro:arg name="l_specific_angle_btw_legs" default="0,180,0,0,10,0" doc=""/>
+    <xacro:arg name="r_specific_angle_btw_legs" default="0,0,5,0,0,0" doc=""/>
     <!-- segmentation -->
     <xacro:arg name="segment_dof" default="2" doc="possible '0','1up','1side','2'"/>
@@ -40,8 +42,8 @@
     <xacro:property name="leg_height" value="$(arg leg_height)"/>
     <xacro:if value="${leg_height == 1}">
-        <xacro:property name="leg_height" value="${0.07}"/>
+        <xacro:property name="leg_height_size" value="${0.07}"/>
     </xacro:if>
     <xacro:if value="${leg_height == 0}">
-        <xacro:property name="leg_height" value="${0.055}"/>
+        <xacro:property name="leg_height_size" value="${0.055}"/>
     </xacro:if>
     <!-- angle between legs -->
@@ -50,8 +52,8 @@
         <xacro:property name="l_specific_angle_btw_legs" value="$(arg l_specific_angle_btw_legs)"/>
         <xacro:property name="r_specific_angle_btw_legs" value="$(arg r_specific_angle_btw_legs)"/>
-        <xacro:property name="offset_btw_legs_wave" value="0"/>
     </xacro:if>
     <xacro:if value="${str(angle_btw_legs) != 'specific'}">
-        <xacro:property name="offset_btw_legs_wave" value="$(arg offset_btw_legs_wave)"/>
+        <xacro:property name="angle_for_0_l_leg" value="$(arg angle_for_0_l_leg)"/>
+        <xacro:property name="angle_for_0_r_leg" default="$(arg angle_for_0_r_leg)"/>
     </xacro:if>
     <!-- segmentation -->
@@ -60,6 +62,7 @@
     <xacro:property name="side_segment_angle" value="$(arg side_segment_angle)"/>
     <!-- Needed constants-variables -->
-    <xacro:property name="dist_btw_legs" value="${0.13}"/>
+    <xacro:property name="dist_btw_legs" value="${0.11}"/>
     <xacro:property name="dist_btw_body_origins" value="${0.554}"/>
+    <xacro:property name="leg_thickness" value="${0.004}"/>
     <xacro:property name="dist_body_1_bridge_1" value="${0.247}"/>
     <xacro:property name="dist_bridge_1_bridge_2" value="${0.03}"/>

File: strirus_robot_description/urdf/strirus_gamma_body_bridge.xacro (robot description, xacro)
@@ -6,5 +6,5 @@
         <parent link="base_footprint"/>
         <child link="body_1_part"/>
-        <origin rpy="0  0  0" xyz="0 0 ${leg_height}"/>
+        <origin rpy="0  0  0" xyz="0 0 ${leg_height_size}"/>
     </joint>
     <!-- /////////////// -->
@@ -178,5 +178,5 @@
             <child link="bridge_2_part"/>
             <origin rpy="0       0      0" xyz="${dist_bridge_1_bridge_2} 0 ${0}"/>
-            <axis xyz="0 1  0"/>
+            <axis xyz="0 -1  0"/>
             <limit effort="30" lower="${-deg2rad*75}" upper="${deg2rad*75}" velocity="5"/>
             <joint_properties damping="0.0" friction="0.0"/>
@@ -188,5 +188,5 @@
             <child link="bridge_1_part"/>
             <origin rpy="0       0      0" xyz="${dist_body_1_bridge_1} 0 ${0}"/>
-            <axis xyz="0 0  1"/>
+            <axis xyz="0 0  -1"/>
             <limit effort="30" lower="${-deg2rad*15}" upper="${deg2rad*15}" velocity="5"/>
             <joint_properties damping="0.0" friction="0.0"/>

File: strirus_robot_description/urdf/strirus_gamma_legs.xacro (robot description, xacro)
@@ -1,3 +1,117 @@
 <?xml version="1.0"?>
 <robot xmlns:xacro="http://www.ros.org/wiki/xacro">
+    <!--
+            <xacro:property name="angle_for_0_l_leg" value="${angle_for_0_l_leg * deg2rad}"/>
+            <xacro:property name="angle_btw_legs" value="${angle_btw_legs * deg2rad}"/> -->
+    <xacro:macro name="leg" params="prefix num side cur_ang">
+        <!-- 		<xacro:property name="angle_coeff_left" value="${(angle_for_0_l_leg + angle_btw_legs * num) % 360 * deg2rad}" />
+                <xacro:property name="angle_coeff_right" value="${-(angle_btw_legs * num) % 360 * deg2rad}" /> -->
+        <link name="leg_${prefix}_${num}">
+            <inertial>
+                <xacro:if value="${leg_height == 0}">
+                    <mass value="${0.010307884}"/>
+                    <xacro:if value="${prefix == 'left'}">
+                        <origin rpy="${0} 0 0" xyz="${-0.008963344} ${0} ${-0.020168668}"/>
+                    </xacro:if>
+                    <xacro:if value="${prefix == 'right'}">
+                        <origin rpy="${0} 0 0" xyz="${-0.008963344} ${0} ${-0.020168668}"/>
+                    </xacro:if>
+                    <inertia
+                            ixx="0.000004032" ixy="0" ixz="0.000000712"
+                            iyy="0.000004993" iyz="0"
+                            izz="0.000001071"/>
+                </xacro:if>
+                <xacro:if value="${leg_height == 1}">
+                    <mass value="${0.012706347}"/>
+                    <xacro:if value="${prefix == 'left'}">
+                        <origin rpy="${0} 0 0" xyz="${-0.013348671} ${0} ${-0.027584119}"/>
+                    </xacro:if>
+                    <xacro:if value="${prefix == 'right'}">
+                        <origin rpy="${0} 0 0" xyz="${-0.013348671} ${0} ${-0.027584119}"/>
+                    </xacro:if>
+                    <inertia
+                            ixx="0.000007895" ixy="0" ixz="0.000001300"
+                            iyy="0.000009763" iyz="0"
+                            izz="0.000002004"/>
+                </xacro:if>
+            </inertial>
+            <collision>
+                <origin rpy="0  0  0" xyz="0 0 0"/>
+                <geometry>
+                    <xacro:if value="${leg_height == 0}">
+                        <mesh filename="package://strirus_cad_design/stl/collision/leg_55.stl" scale="1 1 1"/>
+                    </xacro:if>
+                    <xacro:if value="${leg_height == 1}">
+                        <mesh filename="package://strirus_cad_design/stl/collision/leg_70.stl" scale="1 1 1"/>
+                    </xacro:if>
+                </geometry>
+            </collision>
+            <visual>
+                <origin rpy="0  0  0" xyz="0 0 0"/>
+                <geometry>
+                    <xacro:if value="${leg_height == 0}">
+                        <mesh filename="package://strirus_cad_design/stl/visual/leg_55.stl" scale="1 1 1"/>
+                    </xacro:if>
+                    <xacro:if value="${leg_height == 1}">
+                        <mesh filename="package://strirus_cad_design/stl/visual/leg_70.stl" scale="1 1 1"/>
+                    </xacro:if>
+                </geometry>
+                <material name="white"/>
+            </visual>
+        </link>
+        <joint name="leg_${prefix}_${num}_revolute_joint" type="revolute">
+            <child link="leg_${prefix}_${num}"/>
+            <xacro:if value="${not(num >= amount_of_legs_one_part)}">
+                <parent link="body_1_part"/>
+            	<xacro:if value="${num % 2 and omni_angle == 0}">
+                	<origin rpy="0       0      0"
+                    	    xyz="${dist_btw_legs * (num % amount_of_legs_one_part)} ${0.1555*side}  ${0}"/>
+            	</xacro:if>
+            	<xacro:if value="${not (num % 2) and omni_angle == 0}">
+                	<origin rpy="0       0      0"
+                    	    xyz="${dist_btw_legs * (num % amount_of_legs_one_part)} ${0.1395*side}  ${0}"/>
+            	</xacro:if>
+            	<xacro:if value="${omni_angle != 0}">
+                	<origin rpy="0       0      0"
+                    	    xyz="${-leg_x_offset + dist_btw_legs * (num % amount_of_legs_one_part)} ${leg_y_offset*side}  ${0}"/>
+           		 </xacro:if>
+        </xacro:if>
+            <xacro:if value="${num >= amount_of_legs_one_part}">
+                <parent link="body_2_part"/>
+            	<xacro:if value="${num % 2 and omni_angle == 0}">
+                	<origin rpy="0       0      0"
+                    	    xyz="${dist_body_2_leg_count_point - dist_btw_legs * (num % amount_of_legs_one_part)} ${0.1555*side}  ${0}"/>
+            	</xacro:if>
+            	<xacro:if value="${not (num % 2) and omni_angle == 0}">
+                	<origin rpy="0       0      0"
+                    	    xyz="${dist_body_2_leg_count_point - dist_btw_legs * (num % amount_of_legs_one_part)} ${0.1395*side}  ${0}"/>
+            	</xacro:if>
+            	<xacro:if value="${omni_angle != 0}">
+                	<origin rpy="0       0      0"
+                    	    xyz="${leg_x_offset + dist_body_2_leg_count_point - dist_btw_legs * (num % amount_of_legs_one_part)} ${leg_y_offset*side}  ${0}"/>
+           		 </xacro:if>
+        </xacro:if>
+            <axis xyz="0 -1  0"/>
+            <limit effort="30" lower="-1e+100" upper="1e+100" velocity="3.0"/>
+            <joint_properties damping="0.0" friction="0.0"/>
+        </joint>
+    </xacro:macro>
+    <xacro:if value="${str(angle_btw_legs) == 'specific'}">
+        <xacro:property name="angle_sec_l_leg" value="${l_specific_angle_btw_legs.split(',')}"/>
+        <xacro:property name="angle_sec_r_leg" value="${r_specific_angle_btw_legs.split(',')}"/>
+    </xacro:if>
+    <xacro:if value="${str(angle_btw_legs) != 'specific'}">
+        <xacro:property name="range05" value="${[0,1,2,3,4,5]}"/>
+        <xacro:property name="angle_sec_l_leg" value="${[(angle_for_0_l_leg + i * angle_btw_legs) for i in range05]}"/>
+        <xacro:property name="angle_sec_r_leg" value="${[(angle_for_0_r_leg + i * angle_btw_legs) for i in range05]}"/>
+    </xacro:if>
+    <!-- create needed number of legs (is implemented by recurcion) -->
+    <xacro:macro name="create_legs" params="prefix side number angle_sec">
+        <xacro:leg prefix="${prefix}" num="${number}" side="${side}" cur_ang="${angle_sec[number]}"/>
+        <xacro:if value="${number}">
+            <xacro:create_legs number="${number-1}" prefix="${prefix}" side="${side}" angle_sec="${angle_sec}"/>
+        </xacro:if>
+    </xacro:macro>
+    <xacro:create_legs prefix="left" side="1" number="${number_of_legs}" angle_sec="${angle_sec_l_leg}"/>
+    <xacro:create_legs prefix="right" side="-1" number="${number_of_legs}" angle_sec="${angle_sec_r_leg}"/>
 </robot>
