Commit message: Basic leg functionality were added, code refactoring is needed

File: strirus_robot_description/urdf/strirus_gamma.urdf (robot description, URDF)
Before this commit: robot strirus_gamma, 17 links, 16 joints
Links:
- link body_1_part: geometry collision mesh filename=package://strirus_cad_design/stl/collision/body_1_15_part.s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 scale=1 1 1; visual mesh filename=package://strirus_cad_design/stl/visual/body_1_15_part.stl scale=1 1 1
- link body_2_part: geometry collision mesh filename=package://strirus_cad_design/stl/collision/body_2_15_part.s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 scale=1 1 1; visual mesh filename=package://strirus_cad_design/stl/visual/body_2_15_part.stl scale=1 1 1
- link leg_left_0: mass 0.010307884 -> 0.012706347; geometry collision mesh filename=package://strirus_cad_design/stl/collision/leg_70.stl scale=1 1 1; visual mesh filename=package://strirus_cad_design/stl/visual/leg_70.stl scale=1 1 1
- link leg_left_1: mass 0.010307884 -> 0.012706347; geometry collision mesh filename=package://strirus_cad_design/stl/collision/leg_70.stl scale=1 1 1; visual mesh filename=package://strirus_cad_design/stl/visual/leg_70.stl scale=1 1 1
- link leg_left_2: mass 0.010307884 -> 0.012706347; geometry collision mesh filename=package://strirus_cad_design/stl/collision/leg_70.stl scale=1 1 1; visual mesh filename=package://strirus_cad_design/stl/visual/leg_70.stl scale=1 1 1
- link leg_left_3: mass 0.010307884 -> 0.012706347; geometry collision mesh filename=package://strirus_cad_design/stl/collision/leg_70.stl scale=1 1 1; visual mesh filename=package://strirus_cad_design/stl/visual/leg_70.stl scale=1 1 1
- link leg_left_4: mass 0.010307884 -> 0.012706347; geometry collision mesh filename=package://strirus_cad_design/stl/collision/leg_70.stl scale=1 1 1; visual mesh filename=package://strirus_cad_design/stl/visual/leg_70.stl scale=1 1 1
- link leg_left_5: mass 0.010307884 -> 0.012706347; geometry collision mesh filename=package://strirus_cad_design/stl/collision/leg_70.stl scale=1 1 1; visual mesh filename=package://strirus_cad_design/stl/visual/leg_70.stl scale=1 1 1
- link leg_right_0: mass 0.010307884 -> 0.012706347; geometry collision mesh filename=package://strirus_cad_design/stl/collision/leg_70.stl scale=1 1 1; visual mesh filename=package://strirus_cad_design/stl/visual/leg_70.stl scale=1 1 1
- link leg_right_1: mass 0.010307884 -> 0.012706347; geometry collision mesh filename=package://strirus_cad_design/stl/collision/leg_70.stl scale=1 1 1; visual mesh filename=package://strirus_cad_design/stl/visual/leg_70.stl scale=1 1 1
- link leg_right_2: mass 0.010307884 -> 0.012706347; geometry collision mesh filename=package://strirus_cad_design/stl/collision/leg_70.stl scale=1 1 1; visual mesh filename=package://strirus_cad_design/stl/visual/leg_70.stl scale=1 1 1
- link leg_right_3: mass 0.010307884 -> 0.012706347; geometry collision mesh filename=package://strirus_cad_design/stl/collision/leg_70.stl scale=1 1 1; visual mesh filename=package://strirus_cad_design/stl/visual/leg_70.stl scale=1 1 1
- link leg_right_4: mass 0.010307884 -> 0.012706347; geometry collision mesh filename=package://strirus_cad_design/stl/collision/leg_70.stl scale=1 1 1; visual mesh filename=package://strirus_cad_design/stl/visual/leg_70.stl scale=1 1 1
- link leg_right_5: mass 0.010307884 -> 0.012706347; geometry collision mesh filename=package://strirus_cad_design/stl/collision/leg_70.stl scale=1 1 1; visual mesh filename=package://strirus_cad_design/stl/visual/leg_70.stl scale=1 1 1
Joints:
- joint base_footprint_body_1_part_fixed: origin xyz=0 0 0.055 rpy=0  0  0 -> xyz=0 0 0.07 rpy=0  0  0
- joint body_1_part_bridge_1_part_revolute: origin xyz=0.247 0 0 rpy=0       0      0 -> xyz=0.247 0 0 rpy=0       0      -0.0
- joint bridge_1_part_bridge_2_part_revolute: origin xyz=0.03 0 0 rpy=0       0      0 -> xyz=0.03 0 0 rpy=0       -0.0      0
- joint leg_left_0_revolute_joint: axis 0 1  0 -> 0 -1  0; origin xyz=0.0 0.1345  0 rpy=0       0      0 -> xyz=-0.007893980876 0.1594607377  0 rpy=0       0.0        0.261799387799
- joint leg_left_1_revolute_joint: axis 0 1  0 -> 0 -1  0; origin xyz=0.13 0.1515  0 rpy=0       0      0 -> xyz=0.098106019124 0.1594607377  0 rpy=0       3.14159265359        0.261799387799
- joint leg_left_2_revolute_joint: axis 0 1  0 -> 0 -1  0; origin xyz=0.26 0.1345  0 rpy=0       0      0 -> xyz=0.204106019124 0.1594607377  0 rpy=0       0.0        0.261799387799
- joint leg_left_3_revolute_joint: axis 0 1  0 -> 0 -1  0; origin xyz=0.247 0.1515  0 rpy=0       0      0 -> xyz=0.254893980876 0.1594607377  0 rpy=0       0.0        -0.261799387799
- joint leg_left_4_revolute_joint: axis 0 1  0 -> 0 -1  0; origin xyz=0.117 0.1345  0 rpy=0       0      0 -> xyz=0.148893980876 0.1594607377  0 rpy=0       0.174532925199        -0.261799387799
- joint leg_left_5_revolute_joint: axis 0 1  0 -> 0 -1  0; origin xyz=-0.013 0.1515  0 rpy=0       0      0 -> xyz=0.042893980876 0.1594607377  0 rpy=0       0.0        -0.261799387799
- joint leg_right_0_revolute_joint: axis 0 1  0 -> 0 -1  0; origin xyz=0.0 -0.1345  0 rpy=0       0      0 -> xyz=-0.007893980876 -0.1594607377  0 rpy=0       0.0        -0.261799387799
- joint leg_right_1_revolute_joint: axis 0 1  0 -> 0 -1  0; origin xyz=0.13 -0.1515  0 rpy=0       0      0 -> xyz=0.098106019124 -0.1594607377  0 rpy=0       0.0        -0.261799387799
- joint leg_right_2_revolute_joint: axis 0 1  0 -> 0 -1  0; origin xyz=0.26 -0.1345  0 rpy=0       0      0 -> xyz=0.204106019124 -0.1594607377  0 rpy=0       0.0872664625997        -0.261799387799
- joint leg_right_3_revolute_joint: axis 0 1  0 -> 0 -1  0; origin xyz=0.247 -0.1515  0 rpy=0       0      0 -> xyz=0.254893980876 -0.1594607377  0 rpy=0       0.0        0.261799387799
- joint leg_right_4_revolute_joint: axis 0 1  0 -> 0 -1  0; origin xyz=0.117 -0.1345  0 rpy=0       0      0 -> xyz=0.148893980876 -0.1594607377  0 rpy=0       0.0        0.261799387799
- joint leg_right_5_revolute_joint: axis 0 1  0 -> 0 -1  0; origin xyz=-0.013 -0.1515  0 rpy=0       0      0 -> xyz=0.042893980876 -0.1594607377  0 rpy=0       0.0        0.261799387799

File: strirus_robot_description/urdf/strirus_gamma.xacro (robot description, xacro)
@@ -18,7 +18,7 @@
     <xacro:arg name="leg_fancy_physics" default="0" doc="0 - no, 1 - yes"/>
     <!-- omni-directional -->
-    <xacro:arg name="omni_angle" default="0" doc="possible angles 0,15,30,45"/>
+    <xacro:arg name="omni_angle" default="15" doc="possible angles 0,15,30,45"/>
     <!-- leg size -->
-    <xacro:arg name="leg_height" default="0" doc="0 - 55, 1 - 70"/>
+    <xacro:arg name="leg_height" default="1" doc="0 - 55, 1 - 70"/>
     <!-- angle between legs -->
     <xacro:arg name="angle_btw_legs" default="specific"
@@ -55,5 +55,5 @@
     <xacro:if value="${str(angle_btw_legs) != 'specific'}">
         <xacro:property name="angle_for_0_l_leg" value="$(arg angle_for_0_l_leg)"/>
-        <xacro:property name="angle_for_0_r_leg" default="$(arg angle_for_0_r_leg)"/>
+        <xacro:property name="angle_for_0_r_leg" value="$(arg angle_for_0_r_leg)"/>
     </xacro:if>
     <!-- segmentation -->
@@ -62,5 +62,5 @@
     <xacro:property name="side_segment_angle" value="$(arg side_segment_angle)"/>
     <!-- Needed constants-variables -->
-    <xacro:property name="dist_btw_legs" value="${0.11}"/>
+    <xacro:property name="dist_btw_legs" value="${0.106}"/>
     <xacro:property name="dist_btw_body_origins" value="${0.554}"/>
     <xacro:property name="leg_thickness" value="${0.004}"/>

File: strirus_robot_description/urdf/strirus_gamma_body_bridge.xacro (robot description, xacro)
@@ -163,5 +163,5 @@
             <parent link="body_1_part"/>
             <child link="bridge_1_part"/>
-            <origin rpy="0 0 0" xyz="${dist_body_1_bridge_1} ${0} ${0}"/>
+            <origin rpy="0 ${-deg2rad*up_segment_angle} 0" xyz="${dist_body_1_bridge_1} ${0} ${0}"/>
         </joint>
     </xacro:if>
@@ -170,5 +170,5 @@
             <parent link="bridge_1_part"/>
             <child link="bridge_2_part"/>
-            <origin rpy="0 0 0" xyz="${dist_bridge_1_bridge_2} ${0} ${0}"/>
+            <origin rpy="0 0 ${-deg2rad*side_segment_angle}" xyz="${dist_bridge_1_bridge_2} ${0} ${0}"/>
         </joint>
     </xacro:if>
@@ -177,5 +177,5 @@
             <parent link="bridge_1_part"/>
             <child link="bridge_2_part"/>
-            <origin rpy="0       0      0" xyz="${dist_bridge_1_bridge_2} 0 ${0}"/>
+            <origin rpy="0       ${-deg2rad*up_segment_angle}      0" xyz="${dist_bridge_1_bridge_2} 0 ${0}"/>
             <axis xyz="0 -1  0"/>
             <limit effort="30" lower="${-deg2rad*75}" upper="${deg2rad*75}" velocity="5"/>
@@ -187,5 +187,5 @@
             <parent link="body_1_part"/>
             <child link="bridge_1_part"/>
-            <origin rpy="0       0      0" xyz="${dist_body_1_bridge_1} 0 ${0}"/>
+            <origin rpy="0       0      ${-deg2rad*side_segment_angle}" xyz="${dist_body_1_bridge_1} 0 ${0}"/>
             <axis xyz="0 0  -1"/>
             <limit effort="30" lower="${-deg2rad*15}" upper="${deg2rad*15}" velocity="5"/>

File: strirus_robot_description/urdf/strirus_gamma_legs.xacro (robot description, xacro)
@@ -1,20 +1,22 @@
 <?xml version="1.0"?>
 <robot xmlns:xacro="http://www.ros.org/wiki/xacro">
-    <!--
-            <xacro:property name="angle_for_0_l_leg" value="${angle_for_0_l_leg * deg2rad}"/>
-            <xacro:property name="angle_btw_legs" value="${angle_btw_legs * deg2rad}"/> -->
+            	<xacro:if value="${omni_angle == 15}">
+    				<xacro:property name="leg_x_offset" value="${0.007893980876}"/>
+        	        <xacro:property name="leg_y_offset" value="${0.1594607377}"/>
+           		 </xacro:if>
+             	<xacro:if value="${omni_angle == 30}">
+    				<xacro:property name="leg_x_offset" value="${0.02825}"/>
+        	        <xacro:property name="leg_y_offset" value="${0.1789304353}"/>
+           		 </xacro:if>
+             	<xacro:if value="${omni_angle == 45}">
+    				<xacro:property name="leg_x_offset" value="${0.04631549417}"/>
+        	        <xacro:property name="leg_y_offset" value="${0.1763154942}"/>
+           		 </xacro:if>
     <xacro:macro name="leg" params="prefix num side cur_ang">
-        <!-- 		<xacro:property name="angle_coeff_left" value="${(angle_for_0_l_leg + angle_btw_legs * num) % 360 * deg2rad}" />
-                <xacro:property name="angle_coeff_right" value="${-(angle_btw_legs * num) % 360 * deg2rad}" /> -->
         <link name="leg_${prefix}_${num}">
             <inertial>
                 <xacro:if value="${leg_height == 0}">
                     <mass value="${0.010307884}"/>
-                    <xacro:if value="${prefix == 'left'}">
-                        <origin rpy="${0} 0 0" xyz="${-0.008963344} ${0} ${-0.020168668}"/>
-                    </xacro:if>
-                    <xacro:if value="${prefix == 'right'}">
-                        <origin rpy="${0} 0 0" xyz="${-0.008963344} ${0} ${-0.020168668}"/>
-                    </xacro:if>
+                    <origin rpy="${0} 0 0" xyz="${-0.008963344} ${0} ${-0.020168668}"/>
                     <inertia
                             ixx="0.000004032" ixy="0" ixz="0.000000712"
@@ -24,10 +26,5 @@
                 <xacro:if value="${leg_height == 1}">
                     <mass value="${0.012706347}"/>
-                    <xacro:if value="${prefix == 'left'}">
-                        <origin rpy="${0} 0 0" xyz="${-0.013348671} ${0} ${-0.027584119}"/>
-                    </xacro:if>
-                    <xacro:if value="${prefix == 'right'}">
-                        <origin rpy="${0} 0 0" xyz="${-0.013348671} ${0} ${-0.027584119}"/>
-                    </xacro:if>
+                    <origin rpy="${0} 0 0" xyz="${-0.013348671} ${0} ${-0.027584119}"/>
                     <inertia
                             ixx="0.000007895" ixy="0" ixz="0.000001300"
@@ -65,13 +62,13 @@
                 <parent link="body_1_part"/>
             	<xacro:if value="${num % 2 and omni_angle == 0}">
-                	<origin rpy="0       0      0"
+                	<origin rpy="0       ${deg2rad*cur_ang}        0"
                     	    xyz="${dist_btw_legs * (num % amount_of_legs_one_part)} ${0.1555*side}  ${0}"/>
             	</xacro:if>
             	<xacro:if value="${not (num % 2) and omni_angle == 0}">
-                	<origin rpy="0       0      0"
-                    	    xyz="${dist_btw_legs * (num % amount_of_legs_one_part)} ${0.1395*side}  ${0}"/>
+                	<origin rpy="0       ${deg2rad*cur_ang}        0"
+                    	    xyz="${dist_btw_legs * (num % amount_of_legs_one_part)} ${0.1385*side}  ${0}"/>
             	</xacro:if>
             	<xacro:if value="${omni_angle != 0}">
-                	<origin rpy="0       0      0"
+                	<origin rpy="0       ${deg2rad*cur_ang}        ${deg2rad*omni_angle * side}"
                     	    xyz="${-leg_x_offset + dist_btw_legs * (num % amount_of_legs_one_part)} ${leg_y_offset*side}  ${0}"/>
            		 </xacro:if>
@@ -80,13 +77,13 @@
                 <parent link="body_2_part"/>
             	<xacro:if value="${num % 2 and omni_angle == 0}">
-                	<origin rpy="0       0      0"
+                	<origin rpy="0       ${deg2rad*cur_ang}      0"
                     	    xyz="${dist_body_2_leg_count_point - dist_btw_legs * (num % amount_of_legs_one_part)} ${0.1555*side}  ${0}"/>
             	</xacro:if>
             	<xacro:if value="${not (num % 2) and omni_angle == 0}">
-                	<origin rpy="0       0      0"
-                    	    xyz="${dist_body_2_leg_count_point - dist_btw_legs * (num % amount_of_legs_one_part)} ${0.1395*side}  ${0}"/>
+                	<origin rpy="0       ${deg2rad*cur_ang}        0"
+                    	    xyz="${dist_body_2_leg_count_point - dist_btw_legs * (num % amount_of_legs_one_part)} ${0.1385*side}  ${0}"/>
             	</xacro:if>
             	<xacro:if value="${omni_angle != 0}">
-                	<origin rpy="0       0      0"
+                	<origin rpy="0       ${deg2rad*cur_ang}        ${-deg2rad*omni_angle * side}"
                     	    xyz="${leg_x_offset + dist_body_2_leg_count_point - dist_btw_legs * (num % amount_of_legs_one_part)} ${leg_y_offset*side}  ${0}"/>
            		 </xacro:if>
