Commit message: code was refactored, more fancy features were added. It is needed to solve the problem with angle legs (problem with segment angles were solved)

File: strirus_robot_description/urdf/strirus_gamma.urdf (robot description, URDF)
Before this commit: robot strirus_gamma, 17 links, 16 joints
Joints:
- removed joint body_1_part_bridge_1_part_revolute
- removed joint bridge_1_part_bridge_2_part_revolute
- added joint segment_side_revolute: type revolute, parent body_1_part, child bridge_1_part, origin xyz=0.247 0 0 rpy=0 0 -0.0, axis 0 0  -1, limit lower=-0.261799387799 upper=0.261799387799 effort=5 velocity=0.5
- added joint segment_up_revolute: type revolute, parent bridge_1_part, child bridge_2_part, origin xyz=0.03 0 0 rpy=0 -0.0 0, axis 0 -1  0, limit lower=-1.308996939 upper=1.308996939 effort=5 velocity=0.5
- joint leg_left_0_revolute_joint: limit lower=-1e+100 upper=1e+100 effort=30 velocity=3.0 -> lower=-1e+100 upper=1e+100 effort=1.5 velocity=3.0
- joint leg_left_1_revolute_joint: limit lower=-1e+100 upper=1e+100 effort=30 velocity=3.0 -> lower=-1e+100 upper=1e+100 effort=1.5 velocity=3.0; origin xyz=0.098106019124 0.1594607377  0 rpy=0       3.14159265359        0.261799387799 -> xyz=0.098106019124 0.1594607377  0 rpy=0       2.09439510239        0.261799387799
- joint leg_left_2_revolute_joint: limit lower=-1e+100 upper=1e+100 effort=30 velocity=3.0 -> lower=-1e+100 upper=1e+100 effort=1.5 velocity=3.0; origin xyz=0.204106019124 0.1594607377  0 rpy=0       0.0        0.261799387799 -> xyz=0.204106019124 0.1594607377  0 rpy=0       4.18879020479        0.261799387799
- joint leg_left_3_revolute_joint: limit lower=-1e+100 upper=1e+100 effort=30 velocity=3.0 -> lower=-1e+100 upper=1e+100 effort=1.5 velocity=3.0
- joint leg_left_4_revolute_joint: limit lower=-1e+100 upper=1e+100 effort=30 velocity=3.0 -> lower=-1e+100 upper=1e+100 effort=1.5 velocity=3.0; origin xyz=0.148893980876 0.1594607377  0 rpy=0       0.174532925199        -0.261799387799 -> xyz=0.148893980876 0.1594607377  0 rpy=0       2.09439510239        -0.261799387799
- joint leg_left_5_revolute_joint: limit lower=-1e+100 upper=1e+100 effort=30 velocity=3.0 -> lower=-1e+100 upper=1e+100 effort=1.5 velocity=3.0; origin xyz=0.042893980876 0.1594607377  0 rpy=0       0.0        -0.261799387799 -> xyz=0.042893980876 0.1594607377  0 rpy=0       4.18879020479        -0.261799387799
- joint leg_right_0_revolute_joint: limit lower=-1e+100 upper=1e+100 effort=30 velocity=3.0 -> lower=-1e+100 upper=1e+100 effort=1.5 velocity=3.0
- joint leg_right_1_revolute_joint: limit lower=-1e+100 upper=1e+100 effort=30 velocity=3.0 -> lower=-1e+100 upper=1e+100 effort=1.5 velocity=3.0; origin xyz=0.098106019124 -0.1594607377  0 rpy=0       0.0        -0.261799387799 -> xyz=0.098106019124 -0.1594607377  0 rpy=0       2.09439510239        -0.261799387799
- joint leg_right_2_revolute_joint: limit lower=-1e+100 upper=1e+100 effort=30 velocity=3.0 -> lower=-1e+100 upper=1e+100 effort=1.5 velocity=3.0; origin xyz=0.204106019124 -0.1594607377  0 rpy=0       0.0872664625997        -0.261799387799 -> xyz=0.204106019124 -0.1594607377  0 rpy=0       4.18879020479        -0.261799387799
- joint leg_right_3_revolute_joint: limit lower=-1e+100 upper=1e+100 effort=30 velocity=3.0 -> lower=-1e+100 upper=1e+100 effort=1.5 velocity=3.0
- joint leg_right_4_revolute_joint: limit lower=-1e+100 upper=1e+100 effort=30 velocity=3.0 -> lower=-1e+100 upper=1e+100 effort=1.5 velocity=3.0; origin xyz=0.148893980876 -0.1594607377  0 rpy=0       0.0        0.261799387799 -> xyz=0.148893980876 -0.1594607377  0 rpy=0       2.09439510239        0.261799387799
- joint leg_right_5_revolute_joint: limit lower=-1e+100 upper=1e+100 effort=30 velocity=3.0 -> lower=-1e+100 upper=1e+100 effort=1.5 velocity=3.0; origin xyz=0.042893980876 -0.1594607377  0 rpy=0       0.0        0.261799387799 -> xyz=0.042893980876 -0.1594607377  0 rpy=0       4.18879020479        0.261799387799

File: strirus_robot_description/urdf/strirus_gamma.xacro (robot description, xacro)
@@ -14,25 +14,37 @@
     <!-- Xacro arg provides xacro.py file.xacro real_number_of_legs:=12 -->
     <!-- simulation  options-->
-    <xacro:arg name="ideal_motors" default="0" doc="0 - no, 1 - yes"/>
-    <xacro:arg name="ideal_segment_joint" default="0" doc="0 - no, 1 - yes"/>
-    <xacro:arg name="leg_fancy_physics" default="0" doc="0 - no, 1 - yes"/>
+    <!-- doc="0 - no, 1 - yes" -->
+    <xacro:arg name="ideal_leg_motors" default="1"/>
+    <!-- doc="0 - no, 1 - yes" -->
+    <xacro:arg name="ideal_segment_joint" default="1"/>
+    <!-- doc="0 - no, 1 - yes" -->
+    <xacro:arg name="leg_fancy_physics" default="0"/>
     <!-- omni-directional -->
-    <xacro:arg name="omni_angle" default="15" doc="possible angles 0,15,30,45"/>
+    <!-- doc="possible angles 0,15,30,45" -->
+    <xacro:arg name="omni_angle" default="15"/>
     <!-- leg size -->
-    <xacro:arg name="leg_height" default="1" doc="0 - 55, 1 - 70"/>
+    <!--  doc="0 - 55, 1 - 70" -->
+    <xacro:arg name="leg_height" default="1"/>
     <!-- angle between legs -->
-    <xacro:arg name="angle_btw_legs" default="specific"
-               doc="in degrees, or 'specific' for choosing specific angle for each leg (cclock)"/>
-    <xacro:arg name="angle_for_0_l_leg" default="0" doc="in degrees"/>
-    <xacro:arg name="angle_for_0_r_leg" default="4" doc="in degrees"/>
-    <xacro:arg name="l_specific_angle_btw_legs" default="0,180,0,0,10,0" doc=""/>
-    <xacro:arg name="r_specific_angle_btw_legs" default="0,0,5,0,0,0" doc=""/>
+    <!--  doc="in degrees, or 'specific' for choosing specific angle for each leg (cclock)" -->
+    <xacro:arg name="angle_btw_legs" default="120"/>
+    <!-- doc="in degrees" -->
+    <xacro:arg name="angle_for_0_l_leg" default="0"/>
+    <!-- doc="in degrees" -->
+    <xacro:arg name="angle_for_0_r_leg" default="0"/>
+    <!-- any angle sequence -->
+    <xacro:arg name="l_specific_angle_btw_legs" default="0,180,0,0,10,0"/>
+    <!-- any angle sequence -->
+    <xacro:arg name="r_specific_angle_btw_legs" default="0,0,5,0,0,0"/>
     <!-- segmentation -->
-    <xacro:arg name="segment_dof" default="2" doc="possible '0','1up','1side','2'"/>
-    <xacro:arg name="up_segment_angle" default="0" doc="in degrees"/>
-    <xacro:arg name="side_segment_angle" default="0" doc="in degrees"/>
+    <!-- doc="possible '0','1up','1side','2'" -->
+    <xacro:arg name="segment_dof" default="2"/>
+    <!--  doc="in degrees" -->
+    <xacro:arg name="up_segment_angle" default="0"/>
+    <!--  doc="in degrees" -->
+    <xacro:arg name="side_segment_angle" default="0"/>
     <!-- arg to properties with converting to rad if it is needed -->
     <!-- simulation  options-->
-    <xacro:property name="ideal_motors" value="$(arg ideal_motors)"/>
+    <xacro:property name="ideal_leg_motors" value="$(arg ideal_leg_motors)"/>
     <xacro:property name="ideal_segment_joint" value="$(arg ideal_segment_joint)"/>
     <xacro:property name="leg_fancy_physics" value="$(arg leg_fancy_physics)"/>

File: strirus_robot_description/urdf/strirus_gamma_body_bridge.xacro (robot description, xacro)
@@ -8,5 +8,4 @@
         <origin rpy="0  0  0" xyz="0 0 ${leg_height_size}"/>
     </joint>
-    <!-- /////////////// -->
     <xacro:macro name="full_body" params="omni_deg">
         <!-- omni_deg in DEG!! not  in rad -->
@@ -159,36 +158,46 @@
     </link>
     <!-- Joints -->
-     <xacro:if value="${str(segment_dof) == '0' or str(segment_dof) == '1up'}">
-        <joint name="body_1_part_bridge_1_part_fixed" type="fixed">
+    <xacro:if value="${str(segment_dof) == '0' or str(segment_dof) == '1up'}">
+        <joint name="segment_side_fixed" type="fixed">
             <parent link="body_1_part"/>
             <child link="bridge_1_part"/>
-            <origin rpy="0 ${-deg2rad*up_segment_angle} 0" xyz="${dist_body_1_bridge_1} ${0} ${0}"/>
-        </joint>
-    </xacro:if>
-     <xacro:if value="${str(segment_dof) == '0' or str(segment_dof) == '1side'}">
-        <joint name="bridge_1_part_bridge_2_part_fixed" type="fixed">
+            <origin rpy="0 0 ${-deg2rad*side_segment_angle}" xyz="${dist_body_1_bridge_1} ${0} ${0}"/>
+        </joint>
+    </xacro:if>
+    <xacro:if value="${str(segment_dof) == '0' or str(segment_dof) == '1side'}">
+        <joint name="segment_up_fixed" type="fixed">
             <parent link="bridge_1_part"/>
             <child link="bridge_2_part"/>
-            <origin rpy="0 0 ${-deg2rad*side_segment_angle}" xyz="${dist_bridge_1_bridge_2} ${0} ${0}"/>
+            <origin rpy="0 ${-deg2rad*up_segment_angle} 0" xyz="${dist_bridge_1_bridge_2} ${0} ${0}"/>
         </joint>
     </xacro:if>
     <xacro:if value="${str(segment_dof) == '1up' or str(segment_dof) == '2'}">
-        <joint name="bridge_1_part_bridge_2_part_revolute" type="revolute">
+        <joint name="segment_up_revolute" type="revolute">
             <parent link="bridge_1_part"/>
             <child link="bridge_2_part"/>
-            <origin rpy="0       ${-deg2rad*up_segment_angle}      0" xyz="${dist_bridge_1_bridge_2} 0 ${0}"/>
+             <origin rpy="0 ${-deg2rad*up_segment_angle} 0" xyz="${dist_bridge_1_bridge_2} 0 ${0}"/>
             <axis xyz="0 -1  0"/>
-            <limit effort="30" lower="${-deg2rad*75}" upper="${deg2rad*75}" velocity="5"/>
-            <joint_properties damping="0.0" friction="0.0"/>
+            <limit effort="5" lower="${-deg2rad*75}" upper="${deg2rad*75}" velocity="0.5"/>
+            <xacro:if value="${ideal_segment_joint == 1}">
+                <joint_properties damping="0.0" friction="0.0"/>
+            </xacro:if>
+            <xacro:if value="${ideal_segment_joint == 0}">
+                <joint_properties damping="0.0" friction="0.0"/>
+            </xacro:if>
         </joint>
     </xacro:if>
     <xacro:if value="${str(segment_dof) == '1side' or str(segment_dof) == '2'}">
-        <joint name="body_1_part_bridge_1_part_revolute" type="revolute">
+        <joint name="segment_side_revolute" type="revolute">
             <parent link="body_1_part"/>
             <child link="bridge_1_part"/>
-            <origin rpy="0       0      ${-deg2rad*side_segment_angle}" xyz="${dist_body_1_bridge_1} 0 ${0}"/>
+            <origin rpy="0 0 ${-deg2rad*side_segment_angle}" xyz="${dist_body_1_bridge_1} 0 ${0}"/>
             <axis xyz="0 0  -1"/>
-            <limit effort="30" lower="${-deg2rad*15}" upper="${deg2rad*15}" velocity="5"/>
-            <joint_properties damping="0.0" friction="0.0"/>
+            <limit effort="5" lower="${-deg2rad*15}" upper="${deg2rad*15}" velocity="0.5"/>
+            <xacro:if value="${ideal_segment_joint == 1}">
+                <joint_properties damping="0.0" friction="0.0"/>
+            </xacro:if>
+            <xacro:if value="${ideal_segment_joint == 0}">
+                <joint_properties damping="0.0" friction="0.0"/>
+            </xacro:if>
         </joint>
     </xacro:if>

File: strirus_robot_description/urdf/strirus_gamma_legs.xacro (robot description, xacro)
@@ -1,16 +1,16 @@
 <?xml version="1.0"?>
 <robot xmlns:xacro="http://www.ros.org/wiki/xacro">
-            	<xacro:if value="${omni_angle == 15}">
-    				<xacro:property name="leg_x_offset" value="${0.007893980876}"/>
-        	        <xacro:property name="leg_y_offset" value="${0.1594607377}"/>
-           		 </xacro:if>
-             	<xacro:if value="${omni_angle == 30}">
-    				<xacro:property name="leg_x_offset" value="${0.02825}"/>
-        	        <xacro:property name="leg_y_offset" value="${0.1789304353}"/>
-           		 </xacro:if>
-             	<xacro:if value="${omni_angle == 45}">
-    				<xacro:property name="leg_x_offset" value="${0.04631549417}"/>
-        	        <xacro:property name="leg_y_offset" value="${0.1763154942}"/>
-           		 </xacro:if>
+    <xacro:if value="${omni_angle == 15}">
+        <xacro:property name="leg_x_offset" value="${0.007893980876}"/>
+        <xacro:property name="leg_y_offset" value="${0.1594607377}"/>
+    </xacro:if>
+    <xacro:if value="${omni_angle == 30}">
+        <xacro:property name="leg_x_offset" value="${0.02825}"/>
+        <xacro:property name="leg_y_offset" value="${0.1789304353}"/>
+    </xacro:if>
+    <xacro:if value="${omni_angle == 45}">
+        <xacro:property name="leg_x_offset" value="${0.04631549417}"/>
+        <xacro:property name="leg_y_offset" value="${0.1763154942}"/>
+    </xacro:if>
     <xacro:macro name="leg" params="prefix num side cur_ang">
         <link name="leg_${prefix}_${num}">
@@ -61,54 +61,92 @@
             <xacro:if value="${not(num >= amount_of_legs_one_part)}">
                 <parent link="body_1_part"/>
-            	<xacro:if value="${num % 2 and omni_angle == 0}">
-                	<origin rpy="0       ${deg2rad*cur_ang}        0"
-                    	    xyz="${dist_btw_legs * (num % amount_of_legs_one_part)} ${0.1555*side}  ${0}"/>
-            	</xacro:if>
-            	<xacro:if value="${not (num % 2) and omni_angle == 0}">
-                	<origin rpy="0       ${deg2rad*cur_ang}        0"
-                    	    xyz="${dist_btw_legs * (num % amount_of_legs_one_part)} ${0.1385*side}  ${0}"/>
-            	</xacro:if>
-            	<xacro:if value="${omni_angle != 0}">
-                	<origin rpy="0       ${deg2rad*cur_ang}        ${deg2rad*omni_angle * side}"
-                    	    xyz="${-leg_x_offset + dist_btw_legs * (num % amount_of_legs_one_part)} ${leg_y_offset*side}  ${0}"/>
-           		 </xacro:if>
-        </xacro:if>
+                <xacro:if value="${num % 2 and omni_angle == 0}">
+                    <origin rpy="0       ${deg2rad*cur_ang}        0"
+                            xyz="${dist_btw_legs * (num % amount_of_legs_one_part)} ${0.1555*side}  ${0}"/>
+                </xacro:if>
+                <xacro:if value="${not (num % 2) and omni_angle == 0}">
+                    <origin rpy="0       ${deg2rad*cur_ang}        0"
+                            xyz="${dist_btw_legs * (num % amount_of_legs_one_part)} ${0.1385*side}  ${0}"/>
+                </xacro:if>
+                <xacro:if value="${omni_angle != 0}">
+                    <origin rpy="0       ${deg2rad*cur_ang}        ${deg2rad*omni_angle * side}"
+                            xyz="${-leg_x_offset + dist_btw_legs * (num % amount_of_legs_one_part)} ${leg_y_offset*side}  ${0}"/>
+                </xacro:if>
+            </xacro:if>
             <xacro:if value="${num >= amount_of_legs_one_part}">
                 <parent link="body_2_part"/>
-            	<xacro:if value="${num % 2 and omni_angle == 0}">
-                	<origin rpy="0       ${deg2rad*cur_ang}      0"
-                    	    xyz="${dist_body_2_leg_count_point - dist_btw_legs * (num % amount_of_legs_one_part)} ${0.1555*side}  ${0}"/>
-            	</xacro:if>
-            	<xacro:if value="${not (num % 2) and omni_angle == 0}">
-                	<origin rpy="0       ${deg2rad*cur_ang}        0"
-                    	    xyz="${dist_body_2_leg_count_point - dist_btw_legs * (num % amount_of_legs_one_part)} ${0.1385*side}  ${0}"/>
-            	</xacro:if>
-            	<xacro:if value="${omni_angle != 0}">
-                	<origin rpy="0       ${deg2rad*cur_ang}        ${-deg2rad*omni_angle * side}"
-                    	    xyz="${leg_x_offset + dist_body_2_leg_count_point - dist_btw_legs * (num % amount_of_legs_one_part)} ${leg_y_offset*side}  ${0}"/>
-           		 </xacro:if>
+                <xacro:if value="${num % 2 and omni_angle == 0}">
+                    <origin rpy="0       ${deg2rad*cur_ang}      0"
+                            xyz="${dist_body_2_leg_count_point - dist_btw_legs * (num % amount_of_legs_one_part)} ${0.1555*side}  ${0}"/>
+                </xacro:if>
+                <xacro:if value="${not (num % 2) and omni_angle == 0}">
+                    <origin rpy="0       ${deg2rad*cur_ang}        0"
+                            xyz="${dist_body_2_leg_count_point - dist_btw_legs * (num % amount_of_legs_one_part)} ${0.1385*side}  ${0}"/>
+                </xacro:if>
+                <xacro:if value="${omni_angle != 0}">
+                    <origin rpy="0       ${deg2rad*cur_ang}        ${-deg2rad*omni_angle * side}"
+                            xyz="${leg_x_offset + dist_body_2_leg_count_point - dist_btw_legs * (num % amount_of_legs_one_part)} ${leg_y_offset*side}  ${0}"/>
+                </xacro:if>
+            </xacro:if>
+            <axis xyz="0 -1  0"/>
+            <limit effort="1.5" lower="-1e+100" upper="1e+100" velocity="3.0"/>
+            <xacro:if value="${ideal_leg_motors == 1}">
+                <joint_properties damping="0.0" friction="0.0"/>
+            </xacro:if>
+            <xacro:if value="${ideal_leg_motors == 0}">
+                <joint_properties damping="0.0" friction="0.0"/>
+            </xacro:if>
+        </joint>
+        <gazebo reference="leg_${prefix}_${num}">
+            <material>Gazebo/Gray</material>
+        </gazebo>
+        <xacro:if value="${leg_fancy_physics == 1}">
+            <gazebo reference="leg_${prefix}_${num}">
+                <collision>
+                    <surface>
+                        <bounce>
+                            <restitution_coefficient>0</restitution_coefficient>
+                            <threshold>100000</threshold>
+                        </bounce>
+                        <friction>
+                            <ode>
+                                <mu>0.8</mu>
+                                <mu2>0.8</mu2>
+                                <!-- <fdir1>1 0 0 </fdir1> -->
+                                <slip1>0.2</slip1>
+                                <slip2>0.2</slip2>
+                            </ode>
+                        </friction>
+<!--         			<contact>
+                            <ode>
+                                <kp>1e+12</kp>
+                                <kd>1</kd>
+                                <max_vel>0.01</max_vel>
+                                <soft_erp>0.2</soft_erp>
+                                <soft_cfm>0</soft_cfm>
+                            </ode>
+                        </contact> -->
+                    </surface>
+                </collision>
+            </gazebo>
         </xacro:if>
-            <axis xyz="0 -1  0"/>
-            <limit effort="30" lower="-1e+100" upper="1e+100" velocity="3.0"/>
-            <joint_properties damping="0.0" friction="0.0"/>
-        </joint>
     </xacro:macro>
     <xacro:if value="${str(angle_btw_legs) == 'specific'}">
-        <xacro:property name="angle_sec_l_leg" value="${l_specific_angle_btw_legs.split(',')}"/>
-        <xacro:property name="angle_sec_r_leg" value="${r_specific_angle_btw_legs.split(',')}"/>
+        <xacro:property name="angle_seq_l_leg" value="${l_specific_angle_btw_legs.split(',')}"/>
+        <xacro:property name="angle_seq_r_leg" value="${r_specific_angle_btw_legs.split(',')}"/>
     </xacro:if>
     <xacro:if value="${str(angle_btw_legs) != 'specific'}">
         <xacro:property name="range05" value="${[0,1,2,3,4,5]}"/>
-        <xacro:property name="angle_sec_l_leg" value="${[(angle_for_0_l_leg + i * angle_btw_legs) for i in range05]}"/>
-        <xacro:property name="angle_sec_r_leg" value="${[(angle_for_0_r_leg + i * angle_btw_legs) for i in range05]}"/>
+        <xacro:property name="angle_seq_l_leg" value="${[(angle_for_0_l_leg + i * angle_btw_legs) for i in range05]}"/>
+        <xacro:property name="angle_seq_r_leg" value="${[(angle_for_0_r_leg + i * angle_btw_legs) for i in range05]}"/>
     </xacro:if>
     <!-- create needed number of legs (is implemented by recurcion) -->
-    <xacro:macro name="create_legs" params="prefix side number angle_sec">
-        <xacro:leg prefix="${prefix}" num="${number}" side="${side}" cur_ang="${angle_sec[number]}"/>
+    <xacro:macro name="create_legs" params="prefix side number angle_seq">
+        <xacro:leg prefix="${prefix}" num="${number}" side="${side}" cur_ang="${angle_seq[number]}"/>
         <xacro:if value="${number}">
-            <xacro:create_legs number="${number-1}" prefix="${prefix}" side="${side}" angle_sec="${angle_sec}"/>
+            <xacro:create_legs number="${number-1}" prefix="${prefix}" side="${side}" angle_seq="${angle_seq}"/>
         </xacro:if>
     </xacro:macro>
-    <xacro:create_legs prefix="left" side="1" number="${number_of_legs}" angle_sec="${angle_sec_l_leg}"/>
-    <xacro:create_legs prefix="right" side="-1" number="${number_of_legs}" angle_sec="${angle_sec_r_leg}"/>
+    <xacro:create_legs prefix="left" side="1" number="${number_of_legs}" angle_seq="${angle_seq_l_leg}"/>
+    <xacro:create_legs prefix="right" side="-1" number="${number_of_legs}" angle_seq="${angle_seq_r_leg}"/>
 </robot>
