Commit message: imu and tof camera sensors were added

File: strirus_robot_description/urdf/strirus_gamma.urdf (robot description, URDF)
Before this commit: robot strirus_gamma, 17 links, 16 joints
Links:
- added link tof_camera_1
- added link tof_camera_2
Joints:
- added joint body_1_part_tof_camera_1_fixed: type fixed, parent body_1_part, child tof_camera_1, origin xyz=-0.0375 0 0 rpy=0  0  0
- added joint body_2_part_tof_camera_2_fixed: type fixed, parent body_2_part, child tof_camera_2, origin xyz=-0.2845 0 0 rpy=0  0  0
- joint leg_left_0_revolute_joint: limit lower=-1e+100 upper=1e+100 effort=1.5 velocity=3.0 -> lower=-1e+5 upper=1e+5 effort=1.5 velocity=3.0
- joint leg_left_1_revolute_joint: limit lower=-1e+100 upper=1e+100 effort=1.5 velocity=3.0 -> lower=-1e+5 upper=1e+5 effort=1.5 velocity=3.0
- joint leg_left_2_revolute_joint: limit lower=-1e+100 upper=1e+100 effort=1.5 velocity=3.0 -> lower=-1e+5 upper=1e+5 effort=1.5 velocity=3.0
- joint leg_left_3_revolute_joint: limit lower=-1e+100 upper=1e+100 effort=1.5 velocity=3.0 -> lower=-1e+5 upper=1e+5 effort=1.5 velocity=3.0; origin xyz=0.254893980876 0.1594607377  0 rpy=0       0.0        -0.261799387799 -> xyz=0.254893980876 0.1594607377  0 rpy=0       6.28318530718        -0.261799387799
- joint leg_left_4_revolute_joint: limit lower=-1e+100 upper=1e+100 effort=1.5 velocity=3.0 -> lower=-1e+5 upper=1e+5 effort=1.5 velocity=3.0; origin xyz=0.148893980876 0.1594607377  0 rpy=0       2.09439510239        -0.261799387799 -> xyz=0.148893980876 0.1594607377  0 rpy=0       8.37758040957        -0.261799387799
- joint leg_left_5_revolute_joint: limit lower=-1e+100 upper=1e+100 effort=1.5 velocity=3.0 -> lower=-1e+5 upper=1e+5 effort=1.5 velocity=3.0; origin xyz=0.042893980876 0.1594607377  0 rpy=0       4.18879020479        -0.261799387799 -> xyz=0.042893980876 0.1594607377  0 rpy=0       10.471975512        -0.261799387799
- joint leg_right_0_revolute_joint: limit lower=-1e+100 upper=1e+100 effort=1.5 velocity=3.0 -> lower=-1e+5 upper=1e+5 effort=1.5 velocity=3.0
- joint leg_right_1_revolute_joint: limit lower=-1e+100 upper=1e+100 effort=1.5 velocity=3.0 -> lower=-1e+5 upper=1e+5 effort=1.5 velocity=3.0
- joint leg_right_2_revolute_joint: limit lower=-1e+100 upper=1e+100 effort=1.5 velocity=3.0 -> lower=-1e+5 upper=1e+5 effort=1.5 velocity=3.0
- joint leg_right_3_revolute_joint: limit lower=-1e+100 upper=1e+100 effort=1.5 velocity=3.0 -> lower=-1e+5 upper=1e+5 effort=1.5 velocity=3.0; origin xyz=0.254893980876 -0.1594607377  0 rpy=0       0.0        0.261799387799 -> xyz=0.254893980876 -0.1594607377  0 rpy=0       6.28318530718        0.261799387799
- joint leg_right_4_revolute_joint: limit lower=-1e+100 upper=1e+100 effort=1.5 velocity=3.0 -> lower=-1e+5 upper=1e+5 effort=1.5 velocity=3.0; origin xyz=0.148893980876 -0.1594607377  0 rpy=0       2.09439510239        0.261799387799 -> xyz=0.148893980876 -0.1594607377  0 rpy=0       8.37758040957        0.261799387799
- joint leg_right_5_revolute_joint: limit lower=-1e+100 upper=1e+100 effort=1.5 velocity=3.0 -> lower=-1e+5 upper=1e+5 effort=1.5 velocity=3.0; origin xyz=0.042893980876 -0.1594607377  0 rpy=0       4.18879020479        0.261799387799 -> xyz=0.042893980876 -0.1594607377  0 rpy=0       10.471975512        0.261799387799

File: strirus_robot_description/urdf/strirus_gamma.xacro (robot description, xacro)
@@ -93,3 +93,4 @@
     <xacro:include filename="$(find strirus_robot_description)/urdf/strirus_gamma_body_bridge.xacro"/>
     <xacro:include filename="$(find strirus_robot_description)/urdf/strirus_gamma_legs.xacro"/>
+    <xacro:include filename="$(find strirus_robot_description)/urdf/strirus_gamma_gazebo.gazebo"/>
 </robot>

File: strirus_robot_description/urdf/strirus_gamma_body_bridge.xacro (robot description, xacro)
@@ -58,4 +58,18 @@
             </visual>
         </link>
+        <link name="tof_camera_1">
+        </link>
+        <joint name="body_1_part_tof_camera_1_fixed" type="fixed">
+            <parent link="body_1_part"/>
+            <child link="tof_camera_1"/>
+            <origin rpy="0  0  ${pi}" xyz="-0.0375 0 0"/>
+        </joint>
+        <link name="imu_1">
+        </link>
+        <joint name="body_1_part_imu_1_fixed" type="fixed">
+            <parent link="body_1_part"/>
+            <child link="imu_1"/>
+            <origin rpy="0  0  0" xyz="0 0 0"/>
+        </joint>
         <!--body 2 part -->
         <link name="body_2_part">
@@ -107,4 +121,16 @@
         </link>
     </xacro:macro>
+    <link name="tof_camera_2"/>
+    <joint name="body_2_part_tof_camera_2_fixed" type="fixed">
+        <parent link="body_2_part"/>
+        <child link="tof_camera_2"/>
+        <origin rpy="0  0  0" xyz="0.2845 0 0"/>
+    </joint>
+    <link name="imu_2"/>
+    <joint name="body_2_part_imu_2_fixed" type="fixed">
+        <parent link="body_2_part"/>
+        <child link="imu_2"/>
+        <origin rpy="0  0  0" xyz="0.247 0 0"/>
+    </joint>
     <xacro:full_body omni_deg="${omni_angle}"/>
     <!-- bridge part -->
